Commit message: [fix] ステージをURDFインポートだとCollisionが大雑把過ぎて使えな いので、直接USDを扱うように修正 [fix] velocity_pubが横方向の速度を出力しない不具合を修正 [add] 生成するURDFモデルの位置を固定できるオプションを追加 [bug] 生成するURDFモデルの位置を固定にすると、ステージの原点から動かない...

File: colcon_ws/src/sample_robot_description/robots/sample_robot.urdf.xacro (robot description, xacro)
@@ -6,7 +6,7 @@
   <xacro:include filename="$(find sample_robot_description)/urdf/common.xacro"/>
   <xacro:include filename="$(find sample_robot_description)/urdf/base/base.urdf.xacro"/>
-  <xacro:include filename="$(find sample_robot_description)/urdf/wheel/wheel_100mm_light.urdf.xacro"/>
+  <xacro:include filename="$(find sample_robot_description)/urdf/wheel/wheel_100mm.urdf.xacro"/>
   <xacro:include filename="$(find sample_robot_description)/urdf/shooter/shooter.urdf.xacro"/>
-  <xacro:include filename="$(find sample_robot_description)/gazebo/sample_robot.gazebo.xacro"/>
+  <xacro:include filename="$(find sample_robot_description)/isaac/sample_robot.isaac.xacro"/>
   <xacro:include filename="$(find sample_robot_description)/ros2_control/sample_robot.ros2_control.xacro"/>
   <!-- =============== Link & Joint =============== -->
@@ -33,7 +33,9 @@
 	  <origin xyz="0.35 -0.35 0.05" rpy="0 ${pi/2} ${-pi/4}"/>
   </xacro:omni_wheel>
+<!--
   <xacro:shooter_v0 parent="base_link">
 	<origin xyz="0 0 0.35"/>
   </xacro:shooter_v0>
+-->
   <!-- Base -->
   <xacro:base_gazebo_v0/>
@@ -48,13 +50,6 @@
   </joint>
   <link name="camera_link">
-    <visual>
-      <origin xyz="0 0 0" rpy="0 -1.57 0" />
-      <geometry>
-        <cylinder radius="0.01" length="0.01" />
-      </geometry>
-      <material name="white" />
-    </visual>
   </link>
-  <xacro:sample_robot_gazebo prefix=""/>
+  <xacro:sample_robot_isaac prefix=""/>
   <xacro:sample_robot_ros2_control name="sample_robot" use_sim="$(arg use_sim)"/>
 </robot>

File: colcon_ws/src/sample_robot_description/ros2_control/sample_robot.ros2_control.xacro (robot description, xacro)
@@ -10,5 +10,5 @@
         </xacro:if>
         <xacro:if value="${use_sim}">
-          <plugin>gz_ros2_control/GazeboSimSystem</plugin>
+          <plugin>isaac_ros2_control/IsaacSystem</plugin>
         </xacro:if>
       </hardware>
@@ -57,4 +57,5 @@
         <state_interface name="effort"/>
       </joint>
+<!--
       <joint name="shooter_shaft_link_joint">
         <command_interface name="position">
@@ -112,4 +113,5 @@
         <state_interface name="effort"/>
       </joint>
+-->
     </ros2_control>
   </xacro:macro>

File: colcon_ws/src/sample_robot_description/urdf/base/base.urdf.xacro (robot description, xacro)
@@ -23,7 +23,7 @@
                 <origin xyz="0 0 0"/>
                 <mass value="20.0"/>
-                <inertia ixx="0.1" ixy="0" ixz="0"
-                                 iyy="0.1" iyz="0"
-                                 izz="0.1" />
+                <inertia ixx="5" ixy="0" ixz="0"
+                                 iyy="5" iyz="0"
+                                 izz="5" />
           </inertial>
         </link>

Commit message: [add] ディスク射出機の追加

File: colcon_ws/src/sample_robot_description/robots/sample_robot.urdf.xacro (robot description, xacro)
@@ -33,15 +33,9 @@
 	  <origin xyz="0.35 -0.35 0.05" rpy="0 ${pi/2} ${-pi/4}"/>
   </xacro:omni_wheel>
-<!--
   <xacro:shooter_v0 parent="base_link">
-	<origin xyz="0 0 0.35"/>
+	<origin xyz="0 0 0.30"/>
   </xacro:shooter_v0>
--->
   <!-- Base -->
   <xacro:base_gazebo_v0/>
-  <!-- Wheel -->
-  <!--<xacro:wheel_gazebo_v0 prefix="right"/>-->
-  <!--<xacro:wheel_gazebo_v0 prefix="left"/>-->
-  <!--xacro:wheel_gazebo_control_v0 rate="25"/-->
   <joint name="camera_joint" type="fixed">
     <parent link="base_link"/>
@@ -52,4 +46,4 @@
   </link>
   <xacro:sample_robot_isaac prefix=""/>
-  <xacro:sample_robot_ros2_control name="sample_robot" use_sim="$(arg use_sim)"/>
+  <xacro:sample_robot_ros2_control name="$(arg robot_name)" use_sim="$(arg use_sim)"/>
 </robot>

File: colcon_ws/src/sample_robot_description/ros2_control/sample_robot.ros2_control.xacro (robot description, xacro)
@@ -57,28 +57,5 @@
         <state_interface name="effort"/>
       </joint>
-<!--
-      <joint name="shooter_shaft_link_joint">
-        <command_interface name="position">
-          <param name="min">-0.8</param>
-          <param name="max">0.8</param>
-        </command_interface>
-        <state_interface name="position">
-          <param name="initial_value">0.0</param>
-        </state_interface>
-        <state_interface name="velocity"/>
-        <state_interface name="effort"/>
-      </joint>
-      <joint name="shooter_mag_link_joint">
-        <command_interface name="position">
-          <param name="min">0</param>
-          <param name="max">7</param>
-        </command_interface>
-        <state_interface name="position">
-          <param name="initial_value">0.0</param>
-        </state_interface>
-        <state_interface name="velocity"/>
-        <state_interface name="effort"/>
-      </joint>
-      <joint name="shooter_wheel_link_joint">
+      <joint name="shooter_wheel1_link_joint">
         <command_interface name="velocity">
           <param name="min">0</param>
@@ -102,8 +79,8 @@
         <state_interface name="effort"/>
       </joint>
-      <joint name="shooter_wheel3_link_joint">
+      <joint name="shooter_loader_link_joint">
         <command_interface name="velocity">
           <param name="min">0</param>
-          <param name="max">500</param>
+          <param name="max">6</param>
         </command_interface>
         <state_interface name="position">
@@ -113,5 +90,4 @@
         <state_interface name="effort"/>
       </joint>
--->
     </ros2_control>
   </xacro:macro>

File: colcon_ws/src/sample_robot_description/urdf/shooter/shooter.urdf.xacro (robot description, xacro)
@@ -2,95 +2,327 @@
 <robot xmlns:xacro="http://ros.org/wiki/xacro">
   <xacro:macro name="shooter_v0" params="parent *joint_origin">
-        <joint name="shooter_shaft_link_joint" type="continuous">
+        <joint name="shooter_shaft_link_joint" type="fixed">
           <xacro:insert_block name="joint_origin"/>
           <parent link="${parent}"/>
-          <child link="shooter_shaft_link"/>
-          <axis xyz="0 -1 0"/>
-        </joint>
-        <link name="shooter_shaft_link">
-        </link>
-        <joint name="shooter_body_link_joint" type="fixed">
-          <origin rpy="0 0 0" xyz="0 0 0.0925"/>
-          <parent link="shooter_shaft_link"/>
-          <child link="shooter_body_link"/>
-        </joint>
-        <link name="shooter_body_link">
-          <!--
-          <visual>
-                <geometry>
-                  <mesh filename="file://$(find sample_robot_description)/meshes/STL/shooter_body.stl" />
-                </geometry>
-                <origin rpy="${pi/2} 0 ${pi/2}" xyz="0 -0.12 0"/>
-                <material name="white"/>
-          </visual>
-          -->
-          <collision>
-                <geometry>
-                  <mesh filename="file://$(find sample_robot_description)/meshes/STL/shooter_body.stl" />
-                </geometry>
-                <origin rpy="${pi/2} 0 ${pi/2}" xyz="0 -0.12 0"/>
-          </collision>
-          <inertial>
-                <origin xyz="0 0 0"/>
-                <mass value="20.0"/>
-                <inertia ixx="0.1" ixy="0" ixz="0"
-                                 iyy="0.1" iyz="0"
-                                 izz="0.1" />
-          </inertial>
-        </link>
-        <gazebo reference="shooter_body_link">
-          <selfCollide>false</selfCollide>
-          <mu1 value="0.0" />
-          <mu2 value="0.0" />
-          <kp value="30000000.0" />
-          <kd value="50000000.0" />
-        </gazebo>
-        <joint name="shooter_mag_link_joint" type="continuous">
-          <origin rpy="0 0 0" xyz="0 0 0.0"/>
-          <parent link="shooter_body_link"/>
-          <child link="shooter_mag_link"/>
-          <axis xyz="0 1 0"/>
-        </joint>
-        <link name="shooter_mag_link">
-          <visual>
-                <geometry>
-                  <mesh filename="file://$(find sample_robot_description)/meshes/STL/shooter_mag.stl" />
-                </geometry>
-                <origin rpy="0 0 ${pi/2}" xyz="0 0 0"/>
-                <material name="white"/>
-          </visual>
-          <collision>
-                <geometry>
-                  <mesh filename="file://$(find sample_robot_description)/meshes/STL/shooter_mag.stl" />
-                </geometry>
-                <origin rpy="0 0 ${pi/2}" xyz="0 0 0"/>
-          </collision>
-          <inertial>
-                <origin xyz="0 0 0"/>
-                <mass value="1.0"/>
-                <inertia ixx="0.1" ixy="0" ixz="0"
-                                 iyy="0.1" iyz="0"
-                                 izz="0.1" />
-          </inertial>
-        </link>
-        <gazebo reference="shooter_mag_link">
-          <selfCollide>false</selfCollide>
-          <mu1 value="0.0" />
-          <mu2 value="0.0" />
-          <kp value="30000000.0" />
-          <kd value="50000000.0" />
-        </gazebo>
-         <joint name="shooter_wheel_link_joint" type="continuous">
-          <origin rpy="${-pi/2} 0 0" xyz="0.24 0 -0.145"/> <!-- disc pos x 0.18 z -0.0925 -->
-          <parent link="shooter_body_link"/>
-          <child link="shooter_wheel_link"/>
-          <axis xyz="0 0 1"/>
-        </joint>
-        <link name="shooter_wheel_link">
+          <child link="shooter_base_link"/>
+        </joint>
+        <link name="shooter_base_link">
+          <visual>
+                <geometry>
+                  <box size="0.2 0.18 0.08" />
+                </geometry>
+                <material name="gray"/>
+          </visual>
+          <collision>
+                <geometry>
+                  <box size="0.2 0.18 0.08" />
+                </geometry>
+          </collision>
+          <inertial>
+                <origin xyz="0 0 0"/>
+                <mass value="1.0"/>
+                <inertia ixx="0.1" ixy="0" ixz="0"
+                                 iyy="0.1" iyz="0"
+                                 izz="0.1" />
+          </inertial>
+        </link>
+        <joint name="shooter_wall1_link_joint" type="fixed">
+          <origin rpy="0 0 0" xyz="0.0 0.11 0.05"/>
+          <parent link="shooter_base_link"/>
+          <child link="shooter_wall1_link"/>
+        </joint>
+        <link name="shooter_wall1_link">
+          <visual>
+                <geometry>
+                  <box size="0.2 0.02 0.08" />
+                </geometry>
+                <material name="gray"/>
+          </visual>
+          <collision>
+                <geometry>
+                  <box size="0.2 0.02 0.08" />
+                </geometry>
+          </collision>
+          <inertial>
+                <origin xyz="0 0 0"/>
+                <mass value="1.0"/>
+                <inertia ixx="0.1" ixy="0" ixz="0"
+                                 iyy="0.1" iyz="0"
+                                 izz="0.1" />
+          </inertial>
+        </link>
+        <joint name="shooter_wall2_link_joint" type="fixed">
+          <origin rpy="0 0 0" xyz="0.0 -0.11 0.05"/>
+          <parent link="shooter_base_link"/>
+          <child link="shooter_wall2_link"/>
+        </joint>
+        <link name="shooter_wall2_link">
+          <visual>
+                <geometry>
+                  <box size="0.2 0.02 0.08" />
+                </geometry>
+                <material name="gray"/>
+          </visual>
+          <collision>
+                <geometry>
+                  <box size="0.2 0.02 0.08" />
+                </geometry>
+          </collision>
+          <inertial>
+                <origin xyz="0 0 0"/>
+                <mass value="1.0"/>
+                <inertia ixx="0.1" ixy="0" ixz="0"
+                                 iyy="0.1" iyz="0"
+                                 izz="0.1" />
+          </inertial>
+        </link>
+        <joint name="shooter_pole1_link_joint" type="fixed">
+          <origin rpy="0 0 0" xyz="0.07778 0.07778 0.315"/> <!-- disc pos x 0.18 z -0.0925 -->
+          <parent link="shooter_base_link"/>
+          <child link="shooter_pole1_link"/>
+          <axis xyz="0 0 1"/>
+        </joint>
+        <link name="shooter_pole1_link">
+          <visual>
+                <geometry>
+                  <cylinder length="0.5" radius="0.01" />
+                </geometry>
+                <material name="gray"/>
+          </visual>
+          <collision>
+                <geometry>
+                  <cylinder length="0.5" radius="0.01" />
+                </geometry>
+          </collision>
+          <inertial>
+                <origin xyz="0 0 0"/>
+                <mass value="1.0"/>
+                <inertia ixx="0.1" ixy="0" ixz="0"
+                                 iyy="0.1" iyz="0"
+                                 izz="0.1" />
+          </inertial>
+        </link>
+        <joint name="shooter_pole2_link_joint" type="fixed">
+          <origin rpy="0 0 0" xyz="-0.07778 0.07778 0.315"/> <!-- disc pos x 0.18 z -0.0925 -->
+          <parent link="shooter_base_link"/>
+          <child link="shooter_pole2_link"/>
+          <axis xyz="0 0 1"/>
+        </joint>
+        <link name="shooter_pole2_link">
+          <visual>
+                <geometry>
+                  <cylinder length="0.5" radius="0.01" />
+                </geometry>
+                <material name="gray"/>
+          </visual>
+          <collision>
+                <geometry>
+                  <cylinder length="0.5" radius="0.01" />
+                </geometry>
+          </collision>
+          <inertial>
+                <origin xyz="0 0 0"/>
+                <mass value="1.0"/>
+                <inertia ixx="0.1" ixy="0" ixz="0"
+                                 iyy="0.1" iyz="0"
+                                 izz="0.1" />
+          </inertial>
+        </link>
+        <joint name="shooter_pole3_link_joint" type="fixed">
+          <origin rpy="0 0 0" xyz="-0.07778 -0.07778 0.315"/> <!-- disc pos x 0.18 z -0.0925 -->
+          <parent link="shooter_base_link"/>
+          <child link="shooter_pole3_link"/>
+          <axis xyz="0 0 1"/>
+        </joint>
+        <link name="shooter_pole3_link">
+          <visual>
+                <geometry>
+                  <cylinder length="0.5" radius="0.01" />
+                </geometry>
+                <material name="gray"/>
+          </visual>
+          <collision>
+                <geometry>
+                  <cylinder length="0.5" radius="0.01" />
+                </geometry>
+          </collision>
+          <inertial>
+                <origin xyz="0 0 0"/>
+                <mass value="1.0"/>
+                <inertia ixx="0.1" ixy="0" ixz="0"
+                                 iyy="0.1" iyz="0"
+                                 izz="0.1" />
+          </inertial>
+        </link>
+        <joint name="shooter_pole4_link_joint" type="fixed">
+          <origin rpy="0 0 0" xyz="0.07778 -0.07778 0.315"/> <!-- disc pos x 0.18 z -0.0925 -->
+          <parent link="shooter_base_link"/>
+          <child link="shooter_pole4_link"/>
+          <axis xyz="0 0 1"/>
+        </joint>
+        <link name="shooter_pole4_link">
+          <visual>
+                <geometry>
+                  <cylinder length="0.5" radius="0.01" />
+                </geometry>
+                <material name="gray"/>
+          </visual>
+          <collision>
+                <geometry>
+                  <cylinder length="0.5" radius="0.01" />
+                </geometry>
+          </collision>
+          <inertial>
+                <origin xyz="0 0 0"/>
+                <mass value="1.0"/>
+                <inertia ixx="0.1" ixy="0" ixz="0"
+                                 iyy="0.1" iyz="0"
+                                 izz="0.1" />
+          </inertial>
+        </link>
+        <joint name="shooter_pole5_link_joint" type="fixed">
+          <origin rpy="0 0 0" xyz="0.11 0.0 0.365"/> <!-- disc pos x 0.18 z -0.0925 -->
+          <parent link="shooter_base_link"/>
+          <child link="shooter_pole5_link"/>
+          <axis xyz="0 0 1"/>
+        </joint>
+        <link name="shooter_pole5_link">
+          <visual>
+                <geometry>
+                  <cylinder length="0.4" radius="0.01" />
+                </geometry>
+                <material name="gray"/>
+          </visual>
+          <collision>
+                <geometry>
+                  <cylinder length="0.4" radius="0.01" />
+                </geometry>
+          </collision>
+          <inertial>
+                <origin xyz="0 0 0"/>
+                <mass value="1.0"/>
+                <inertia ixx="0.1" ixy="0" ixz="0"
+                                 iyy="0.1" iyz="0"
+                                 izz="0.1" />
+          </inertial>
+        </link>
+        <joint name="shooter_pole6_link_joint" type="fixed">
+          <origin rpy="0 0 0" xyz="-0.11 0.0 0.315"/> <!-- disc pos x 0.18 z -0.0925 -->
+          <parent link="shooter_base_link"/>
+          <child link="shooter_pole6_link"/>
+          <axis xyz="0 0 1"/>
+        </joint>
+        <link name="shooter_pole6_link">
+          <visual>
+                <geometry>
+                  <cylinder length="0.5" radius="0.01" />
+                </geometry>
+                <material name="gray"/>
+          </visual>
+          <collision>
+                <geometry>
+                  <cylinder length="0.5" radius="0.01" />
+                </geometry>
+          </collision>
+          <inertial>
+                <origin xyz="0 0 0"/>
+                <mass value="1.0"/>
+                <inertia ixx="0.1" ixy="0" ixz="0"
+                                 iyy="0.1" iyz="0"
+                                 izz="0.1" />
+          </inertial>
+        </link>
+        <joint name="shooter_pole7_link_joint" type="fixed">
+          <origin rpy="0 0 0" xyz="0.0 0.11 0.315"/> <!-- disc pos x 0.18 z -0.0925 -->
+          <parent link="shooter_base_link"/>
+          <child link="shooter_pole7_link"/>
+          <axis xyz="0 0 1"/>
+        </joint>
+        <link name="shooter_pole7_link">
+          <visual>
+                <geometry>
+                  <cylinder length="0.5" radius="0.01" />
+                </geometry>
+                <material name="gray"/>
+          </visual>
+          <collision>
+                <geometry>
+                  <cylinder length="0.5" radius="0.01" />
+                </geometry>
+          </collision>
+          <inertial>
+                <origin xyz="0 0 0"/>
+                <mass value="1.0"/>
+                <inertia ixx="0.1" ixy="0" ixz="0"
+                                 iyy="0.1" iyz="0"
+                                 izz="0.1" />
+          </inertial>
+        </link>
+        <joint name="shooter_pole8_link_joint" type="fixed">
+          <origin rpy="0 0 0" xyz="0.0 -0.11 0.315"/> <!-- disc pos x 0.18 z -0.0925 -->
+          <parent link="shooter_base_link"/>
+          <child link="shooter_pole8_link"/>
+          <axis xyz="0 0 1"/>
+        </joint>
+        <link name="shooter_pole8_link">
+          <visual>
+                <geometry>
+                  <cylinder length="0.5" radius="0.01" />
+                </geometry>
+                <material name="gray"/>
+          </visual>
+          <collision>
+                <geometry>
+                  <cylinder length="0.5" radius="0.01" />
+                </geometry>
+          </collision>
+          <inertial>
+                <origin xyz="0 0 0"/>
+                <mass value="1.0"/>
+                <inertia ixx="0.1" ixy="0" ixz="0"
+                                 iyy="0.1" iyz="0"
+                                 izz="0.1" />
+          </inertial>
+        </link>
+         <joint name="shooter_loader_link_joint" type="continuous">
+          <origin rpy="0 0 0" xyz="-0.12 0 0.05"/>
+          <parent link="shooter_base_link"/>
+          <child link="shooter_loader_link"/>
+          <axis xyz="0 0 1"/>
+        </joint>
+        <link name="shooter_loader_link">
+          <visual>
+            <origin rpy="0 0 0" xyz="-0.05 0 0.0"/>
+                <geometry>
+                  <box size="0.1 0.04 0.02" />
+                </geometry>
+                <material name="gray"/>
+          </visual>
+          <collision>
+            <origin rpy="0 0 0" xyz="-0.05 0 0.0"/>
+                <geometry>
+                  <box size="0.1 0.04 0.02" />
+                </geometry>
+          </collision>
+          <inertial>
+                <origin xyz="0 0 0"/>
+                <mass value="1.0"/>
+                <inertia ixx="0.1" ixy="0" ixz="0"
+                                 iyy="0.1" iyz="0"
+                                 izz="0.1" />
+          </inertial>
+        </link>
+         <joint name="shooter_wheel1_link_joint" type="continuous">
+          <origin rpy="${-pi/2} 0 0" xyz="0.15 0 0.015"/> <!-- disc pos x 0.18 z -0.0925 -->
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