Commit message: [add] prismatic joint

File: colcon_ws/src/sample_robot_description/urdf/shooter/shooter.urdf.xacro (robot description, xacro)
@@ -285,9 +285,10 @@
           </inertial>
         </link>
-         <joint name="shooter_loader_link_joint" type="continuous">
+         <joint name="shooter_loader_link_joint" type="prismatic">
           <origin rpy="0 0 0" xyz="-0.12 0 0.05"/>
+          <limit lower="0.0" upper="0.2" effort="100" velocity="1.0" />
           <parent link="shooter_base_link"/>
           <child link="shooter_loader_link"/>
-          <axis xyz="0 0 1"/>
+          <axis xyz="1 0 0"/>
         </joint>
         <link name="shooter_loader_link">
@@ -295,5 +296,5 @@
             <origin rpy="0 0 0" xyz="-0.05 0 0.0"/>
                 <geometry>
-                  <box size="0.1 0.04 0.02" />
+                  <box size="0.1 0.1 0.01" />
                 </geometry>
                 <material name="gray"/>
@@ -302,5 +303,5 @@
             <origin rpy="0 0 0" xyz="-0.05 0 0.0"/>
                 <geometry>
-                  <box size="0.1 0.04 0.02" />
+                  <box size="0.1 0.1 0.01" />
                 </geometry>
           </collision>
