Commit message: [upgrade] 射出機周りの摩擦を見直し、威力・安定性を向上

File: colcon_ws/src/flying_disc_description/urdf/common.xacro (robot description, xacro)
@@ -2,21 +2,15 @@
 <robot xmlns:xacro="http://ros.org/wiki/xacro">
   <xacro:macro name="pi" params="3.1415926535897931" />
-  <material name="gray">
-    <color rgba="0.8 0.8 0.8 1.0"/>
-  </material>
   <material name="black">
     <color rgba="0 0 0 1.0"/>
+    <isaac_rigid_body static_friction="0.8" dynamic_friction="0.6"/>
   </material>
   <material name="white">
     <color rgba="1.0 1.0 1.0 1.0"/>
+    <isaac_rigid_body static_friction="0.8" dynamic_friction="0.6"/>
   </material>
   <material name="red">
     <color rgba="1.0 0 0 1.0"/>
-  </material>
-  <material name="light_red">
-    <color rgba="1.0 0.5 0.5 1.0"/>
-  </material>
-  <material name="yellow">
-    <color rgba="0 1.0 1.0 1.0"/>
+    <isaac_rigid_body static_friction="0.8" dynamic_friction="0.6"/>
   </material>
 </robot>

File: colcon_ws/src/flying_disc_description/urdf/flying_disc.urdf.xacro (robot description, xacro)
@@ -32,9 +32,3 @@
     </inertial>
   </link>
-  <gazebo reference="disc_link">
-    <material>Gazebo/White</material>
-    <selfCollide>true</selfCollide>
-    <mu1 value="0.5" />
-    <mu2 value="0.5" />
-  </gazebo>
 </robot>

File: colcon_ws/src/sample_robot_description/ros2_control/sample_robot.ros2_control.xacro (robot description, xacro)
@@ -10,5 +10,8 @@
         </xacro:if>
         <xacro:if value="${use_sim}">
-          <plugin>isaac_ros2_control/IsaacSystem</plugin>
+          <plugin>topic_based_ros2_control/TopicBasedSystem</plugin>
+          <param name="joint_commands_topic">/${name}/joint_command</param>
+          <param name="joint_states_topic">/${name}/joint_states</param>
+          <param name="sum_wrapped_joint_states">true</param>
         </xacro:if>
       </hardware>
@@ -60,5 +63,5 @@
         <command_interface name="velocity">
           <param name="min">0</param>
-          <param name="max">800</param>
+          <param name="max">1600</param>
         </command_interface>
         <state_interface name="position">
@@ -71,5 +74,5 @@
         <command_interface name="velocity">
           <param name="min">0</param>
-          <param name="max">800</param>
+          <param name="max">1600</param>
         </command_interface>
         <state_interface name="position">

File: colcon_ws/src/sample_robot_description/urdf/common.xacro (robot description, xacro)
@@ -3,20 +3,30 @@
   <xacro:macro name="pi" params="3.1415926535897931" />
   <material name="gray">
-    <color rgba="0.8 0.8 0.8 1.0"/>
+    <color rgba="0.6 0.6 0.6 1.0"/>
+    <isaac_rigid_body static_friction="1.0" dynamic_friction="1.0"/>
   </material>
   <material name="black">
     <color rgba="0 0 0 1.0"/>
+    <isaac_rigid_body static_friction="1.0" dynamic_friction="1.0"/>
   </material>
   <material name="white">
     <color rgba="1.0 1.0 1.0 1.0"/>
+    <isaac_rigid_body static_friction="1.0" dynamic_friction="1.0"/>
+  </material>
+  <material name="shooter_unit">
+    <color rgba="0.4 0.4 0.4 1.0"/>
+    <isaac_rigid_body static_friction="0.2" dynamic_friction="0.0"/>
   </material>
   <material name="red">
     <color rgba="1.0 0 0 1.0"/>
+    <isaac_rigid_body static_friction="1.0" dynamic_friction="1.0"/>
   </material>
   <material name="light_red">
     <color rgba="1.0 0.5 0.5 1.0"/>
+    <isaac_rigid_body static_friction="1.0" dynamic_friction="1.0"/>
   </material>
   <material name="yellow">
     <color rgba="0 1.0 1.0 1.0"/>
+    <isaac_rigid_body static_friction="1.0" dynamic_friction="1.0"/>
   </material>
 </robot>

File: colcon_ws/src/sample_robot_description/urdf/shooter/shooter.urdf.xacro (robot description, xacro)
@@ -13,5 +13,5 @@
                   <box size="0.3 0.18 0.08" />
                 </geometry>
-                <material name="gray"/>
+                <material name="shooter_unit"/>
           </visual>
           <collision>
@@ -39,5 +39,5 @@
                   <box size="0.1 0.18 0.04" />
                 </geometry>
-                <material name="gray"/>
+                <material name="shooter_unit"/>
           </visual>
           <collision>
@@ -64,5 +64,5 @@
                   <box size="0.2 0.02 0.08" />
                 </geometry>
-                <material name="gray"/>
+                <material name="shooter_unit"/>
           </visual>
           <collision>
@@ -89,5 +89,5 @@
                   <box size="0.2 0.02 0.08" />
                 </geometry>
-                <material name="gray"/>
+                <material name="shooter_unit"/>
           </visual>
           <collision>
@@ -114,5 +114,5 @@
                   <box size="0.1 0.02 0.08" />
                 </geometry>
-                <material name="gray"/>
+                <material name="shooter_unit"/>
           </visual>
           <collision>
@@ -139,5 +139,5 @@
                   <box size="0.1 0.02 0.08" />
                 </geometry>
-                <material name="gray"/>
+                <material name="shooter_unit"/>
           </visual>
           <collision>
@@ -165,5 +165,5 @@
                   <cylinder length="0.5" radius="0.01" />
                 </geometry>
-                <material name="gray"/>
+                <material name="shooter_unit"/>
           </visual>
           <collision>
@@ -191,5 +191,5 @@
                   <cylinder length="0.5" radius="0.01" />
                 </geometry>
-                <material name="gray"/>
+                <material name="shooter_unit"/>
           </visual>
           <collision>
@@ -217,5 +217,5 @@
                   <cylinder length="0.5" radius="0.01" />
                 </geometry>
-                <material name="gray"/>
+                <material name="shooter_unit"/>
           </visual>
           <collision>
@@ -243,5 +243,5 @@
                   <cylinder length="0.5" radius="0.01" />
                 </geometry>
-                <material name="gray"/>
+                <material name="shooter_unit"/>
           </visual>
           <collision>
@@ -269,5 +269,5 @@
                   <cylinder length="0.45" radius="0.01" />
                 </geometry>
-                <material name="gray"/>
+                <material name="shooter_unit"/>
           </visual>
           <collision>
@@ -295,5 +295,5 @@
                   <cylinder length="0.5" radius="0.01" />
                 </geometry>
-                <material name="gray"/>
+                <material name="shooter_unit"/>
           </visual>
           <collision>
@@ -321,5 +321,5 @@
                   <cylinder length="0.5" radius="0.01" />
                 </geometry>
-                <material name="gray"/>
+                <material name="shooter_unit"/>
           </visual>
           <collision>
@@ -347,5 +347,5 @@
                   <cylinder length="0.5" radius="0.01" />
                 </geometry>
-                <material name="gray"/>
+                <material name="shooter_unit"/>
           </visual>
           <collision>
@@ -375,5 +375,5 @@
                   <box size="0.1 0.1 0.01" />
                 </geometry>
-                <material name="gray"/>
+                <material name="shooter_unit"/>
           </visual>
           <collision>
@@ -392,5 +392,5 @@
         </link>
          <joint name="shooter_wheel1_link_joint" type="continuous">
-          <origin rpy="0 0 0" xyz="0.15 0.13 0.055"/> <!-- disc pos x 0.18 z -0.0925 -->
+          <origin rpy="0 0 0" xyz="0.15 0.12 0.055"/> <!-- disc pos x 0.18 z -0.0925 -->
           <parent link="shooter_base_link"/>
           <child link="shooter_wheel1_link"/>
@@ -418,5 +418,5 @@
         </link>
          <joint name="shooter_wheel2_link_joint" type="continuous">
-          <origin rpy="0 0 0" xyz="0.15 -0.13 0.055"/> <!-- disc pos x 0.18 z -0.0925 -->
+          <origin rpy="0 0 0" xyz="0.15 -0.12 0.055"/> <!-- disc pos x 0.18 z -0.0925 -->
           <parent link="shooter_base_link"/>
           <child link="shooter_wheel2_link"/>

File: colcon_ws/src/sample_robot_description/urdf/wheel/wheel_100mm.urdf.xacro (robot description, xacro)
@@ -7,5 +7,5 @@
       <origin rpy="${pi/2} 0 ${dir}" xyz="${0.0368*cos(dir)} ${0.0368*sin(dir)} 0.0158"/>
       <axis xyz="0 0 1"/>
-      <dynamics damping="0.001"/>
+      <isaac_drive_api stiffness="0" damping="0" joint_friction="0"/>
     </joint>
     <link name="${prefix}_link">
@@ -26,21 +26,4 @@
       </inertial>
     </link>
-    <gazebo reference="${prefix}_link">
-      <mu1 value="2.5" />
-      <mu2 value="2.5" />
-      <kp value="5000.0" />
-      <kd value="10.0" />
-      <material>Gazebo/Black</material>
-    </gazebo>
-    <transmission name="${prefix}_trans">
-      <type>transmission_interface/SimpleTransmission</type>
-      <joint name="${prefix}_joint">
-        <hardwareInterface>hardware_interface/EffortJointInterface</hardwareInterface>
-      </joint>
-      <actuator name="${prefix}_motor">
-        <hardwareInterface>hardware_interface/EffortJointInterface</hardwareInterface>
-        <mechanicalReduction>1</mechanicalReduction>
-      </actuator>
-    </transmission>
   </xacro:macro>
   <xacro:macro name="omni_wheel" params="prefix parent *joint_origin">
@@ -50,16 +33,6 @@
     <xacro:insert_block name="joint_origin"/>
     <axis xyz="0 0 1"/>
-    <dynamics damping="0.7"/>
+    <isaac_drive_api stiffness="0" damping="30000" joint_friction="0"/>
   </joint>
-  <transmission name="${prefix}_shaft_trans">
-    <type>transmission_interface/SimpleTransmission</type>
-    <joint name="${prefix}_shaft_joint">
-      <hardwareInterface>hardware_interface/VelocityJointInterface</hardwareInterface>
-    </joint>
-    <actuator name="${prefix}_shaft_motor">
-      <hardwareInterface>hardware_interface/VelocityJointInterface</hardwareInterface>
-      <mechanicalReduction>1</mechanicalReduction>
-    </actuator>
-  </transmission>
     <link name="${prefix}_housing_link">
       <visual>
