Commit message: [change] ディスクのUSDファイルの中身を参照を使うように修正 [fix] hp_managerが命中する鎧によってHPを回復してしまう不具合を修正 [update] isaac_ros2_utilsを更新 [change] ロボットの操作にイネーブルスイッチが必要ないように変更 [fix] URDFファイルの慣性情報が間違っている部分を修正 [change] ロボットプログラムの立ち上げ順序を変更

File: colcon_ws/src/sample_robot_description/isaac/sample_robot.isaac.xacro (robot description, xacro)
@@ -12,6 +12,6 @@
         <projection>perspective</projection> <!-- perspective or orthgonal -->
         <image>
-           <width>960</width>
-           <height>540</height>
+           <width>640</width>
+           <height>360</height>
         </image>
         <clip>
@@ -19,5 +19,5 @@
           <far>300</far>
         </clip>
-        <update_rate>10.0</update_rate>
+        <update_rate>5.0</update_rate>
       </sensor>
       <sensor name="armor1_link" type="contact">

File: colcon_ws/src/sample_robot_description/robots/sample_robot_1.urdf.xacro (robot description, xacro)
@@ -12,5 +12,13 @@
   <!-- =============== Link & Joint =============== -->
   <!-- Base -->
-  <link name="base_link"/>
+  <link name="base_link">
+    <inertial>
+      <origin xyz="0 0 0"/>
+      <mass value="0.0001"/>
+      <inertia ixx="0.00001" ixy="0" ixz="0"
+                         iyy="0.00001" iyz="0"
+                                 izz="0.00001" />
+    </inertial>
+  </link>
   <xacro:base_v0 parent="base_link">
 	<origin xyz="0 0 0.06"/>
@@ -44,4 +52,11 @@
   </joint>
   <link name="camera_link">
+    <inertial>
+      <origin xyz="0 0 0"/>
+      <mass value="0.0001"/>
+      <inertia ixx="0.00001" ixy="0" ixz="0"
+                         iyy="0.00001" iyz="0"
+                                 izz="0.00001" />
+    </inertial>
   </link>
   <joint name="armor1_joint" type="fixed">
@@ -59,5 +74,5 @@
     <collision>
       <geometry>
-        <box size="0.6 0.6 0.02" />
+        <box size="0.1 0.3 0.3" />
       </geometry>
     </collision>
@@ -84,5 +99,5 @@
     <collision>
       <geometry>
-        <box size="0.6 0.6 0.02" />
+        <box size="0.1 0.3 0.3" />
       </geometry>
     </collision>
@@ -109,5 +124,5 @@
     <collision>
       <geometry>
-        <box size="0.6 0.6 0.02" />
+        <box size="0.1 0.3 0.3" />
       </geometry>
     </collision>
@@ -134,5 +149,5 @@
     <collision>
       <geometry>
-        <box size="0.6 0.6 0.02" />
+        <box size="0.1 0.3 0.3" />
       </geometry>
     </collision>

File: colcon_ws/src/sample_robot_description/robots/sample_robot_2.urdf.xacro (robot description, xacro)
@@ -12,5 +12,13 @@
   <!-- =============== Link & Joint =============== -->
   <!-- Base -->
-  <link name="base_link"/>
+  <link name="base_link">
+    <inertial>
+      <origin xyz="0 0 0"/>
+      <mass value="0.0001"/>
+      <inertia ixx="0.00001" ixy="0" ixz="0"
+                         iyy="0.00001" iyz="0"
+                                 izz="0.00001" />
+    </inertial>
+  </link>
   <xacro:base_v0 parent="base_link">
 	<origin xyz="0 0 0.06"/>
@@ -44,4 +52,11 @@
   </joint>
   <link name="camera_link">
+    <inertial>
+      <origin xyz="0 0 0"/>
+      <mass value="0.0001"/>
+      <inertia ixx="0.00001" ixy="0" ixz="0"
+                         iyy="0.00001" iyz="0"
+                                 izz="0.00001" />
+    </inertial>
   </link>
   <joint name="armor1_joint" type="fixed">
@@ -59,5 +74,5 @@
     <collision>
       <geometry>
-        <box size="0.6 0.6 0.02" />
+        <box size="0.1 0.3 0.3" />
       </geometry>
     </collision>
@@ -84,5 +99,5 @@
     <collision>
       <geometry>
-        <box size="0.6 0.6 0.02" />
+        <box size="0.1 0.3 0.3" />
       </geometry>
     </collision>
@@ -109,5 +124,5 @@
     <collision>
       <geometry>
-        <box size="0.6 0.6 0.02" />
+        <box size="0.1 0.3 0.3" />
       </geometry>
     </collision>
@@ -134,5 +149,5 @@
     <collision>
       <geometry>
-        <box size="0.6 0.6 0.02" />
+        <box size="0.1 0.3 0.3" />
       </geometry>
     </collision>

File: colcon_ws/src/sample_robot_description/robots/sample_robot_3.urdf.xacro (robot description, xacro)
@@ -12,5 +12,13 @@
   <!-- =============== Link & Joint =============== -->
   <!-- Base -->
-  <link name="base_link"/>
+  <link name="base_link">
+    <inertial>
+      <origin xyz="0 0 0"/>
+      <mass value="0.0001"/>
+      <inertia ixx="0.00001" ixy="0" ixz="0"
+                         iyy="0.00001" iyz="0"
+                                 izz="0.00001" />
+    </inertial>
+  </link>
   <xacro:base_v0 parent="base_link">
 	<origin xyz="0 0 0.06"/>
@@ -44,4 +52,11 @@
   </joint>
   <link name="camera_link">
+    <inertial>
+      <origin xyz="0 0 0"/>
+      <mass value="0.0001"/>
+      <inertia ixx="0.00001" ixy="0" ixz="0"
+                         iyy="0.00001" iyz="0"
+                                 izz="0.00001" />
+    </inertial>
   </link>
   <joint name="armor1_joint" type="fixed">
@@ -59,5 +74,5 @@
     <collision>
       <geometry>
-        <box size="0.6 0.6 0.02" />
+        <box size="0.1 0.3 0.3" />
       </geometry>
     </collision>
@@ -84,5 +99,5 @@
     <collision>
       <geometry>
-        <box size="0.6 0.6 0.02" />
+        <box size="0.1 0.3 0.3" />
       </geometry>
     </collision>
@@ -109,5 +124,5 @@
     <collision>
       <geometry>
-        <box size="0.6 0.6 0.02" />
+        <box size="0.1 0.3 0.3" />
       </geometry>
     </collision>
@@ -134,5 +149,5 @@
     <collision>
       <geometry>
-        <box size="0.6 0.6 0.02" />
+        <box size="0.1 0.3 0.3" />
       </geometry>
     </collision>

File: colcon_ws/src/sample_robot_description/robots/sample_robot_4.urdf.xacro (robot description, xacro)
@@ -12,5 +12,13 @@
   <!-- =============== Link & Joint =============== -->
   <!-- Base -->
-  <link name="base_link"/>
+  <link name="base_link">
+    <inertial>
+      <origin xyz="0 0 0"/>
+      <mass value="0.0001"/>
+      <inertia ixx="0.00001" ixy="0" ixz="0"
+                         iyy="0.00001" iyz="0"
+                                 izz="0.00001" />
+    </inertial>
+  </link>
   <xacro:base_v0 parent="base_link">
 	<origin xyz="0 0 0.06"/>
@@ -44,4 +52,11 @@
   </joint>
   <link name="camera_link">
+    <inertial>
+      <origin xyz="0 0 0"/>
+      <mass value="0.0001"/>
+      <inertia ixx="0.00001" ixy="0" ixz="0"
+                         iyy="0.00001" iyz="0"
+                                 izz="0.00001" />
+    </inertial>
   </link>
   <joint name="armor1_joint" type="fixed">

File: colcon_ws/src/sample_robot_description/robots/sample_robot_5.urdf.xacro (robot description, xacro)
@@ -12,5 +12,13 @@
   <!-- =============== Link & Joint =============== -->
   <!-- Base -->
-  <link name="base_link"/>
+  <link name="base_link">
+    <inertial>
+      <origin xyz="0 0 0"/>
+      <mass value="0.0001"/>
+      <inertia ixx="0.00001" ixy="0" ixz="0"
+                         iyy="0.00001" iyz="0"
+                                 izz="0.00001" />
+    </inertial>
+  </link>
   <xacro:base_v0 parent="base_link">
 	<origin xyz="0 0 0.06"/>
@@ -44,4 +52,11 @@
   </joint>
   <link name="camera_link">
+    <inertial>
+      <origin xyz="0 0 0"/>
+      <mass value="0.0001"/>
+      <inertia ixx="0.00001" ixy="0" ixz="0"
+                         iyy="0.00001" iyz="0"
+                                 izz="0.00001" />
+    </inertial>
   </link>
   <joint name="armor1_joint" type="fixed">

File: colcon_ws/src/sample_robot_description/robots/sample_robot_6.urdf.xacro (robot description, xacro)
@@ -12,5 +12,13 @@
   <!-- =============== Link & Joint =============== -->
   <!-- Base -->
-  <link name="base_link"/>
+  <link name="base_link">
+    <inertial>
+      <origin xyz="0 0 0"/>
+      <mass value="0.0001"/>
+      <inertia ixx="0.00001" ixy="0" ixz="0"
+                         iyy="0.00001" iyz="0"
+                                 izz="0.00001" />
+    </inertial>
+  </link>
   <xacro:base_v0 parent="base_link">
 	<origin xyz="0 0 0.06"/>
@@ -44,4 +52,11 @@
   </joint>
   <link name="camera_link">
+    <inertial>
+      <origin xyz="0 0 0"/>
+      <mass value="0.0001"/>
+      <inertia ixx="0.00001" ixy="0" ixz="0"
+                         iyy="0.00001" iyz="0"
+                                 izz="0.00001" />
+    </inertial>
   </link>
   <joint name="armor1_joint" type="fixed">

File: colcon_ws/src/sample_robot_description/robots/sample_robot_7.urdf.xacro (robot description, xacro)
@@ -12,5 +12,13 @@
   <!-- =============== Link & Joint =============== -->
   <!-- Base -->
-  <link name="base_link"/>
+  <link name="base_link">
+    <inertial>
+      <origin xyz="0 0 0"/>
+      <mass value="0.0001"/>
+      <inertia ixx="0.00001" ixy="0" ixz="0"
+                         iyy="0.00001" iyz="0"
+                                 izz="0.00001" />
+    </inertial>
+  </link>
   <xacro:base_v0 parent="base_link">
 	<origin xyz="0 0 0.06"/>
@@ -44,4 +52,11 @@
   </joint>
   <link name="camera_link">
+    <inertial>
+      <origin xyz="0 0 0"/>
+      <mass value="0.0001"/>
+      <inertia ixx="0.00001" ixy="0" ixz="0"
+                         iyy="0.00001" iyz="0"
+                                 izz="0.00001" />
+    </inertial>
   </link>
   <joint name="armor1_joint" type="fixed">

File: colcon_ws/src/sample_robot_description/robots/sample_robot_8.urdf.xacro (robot description, xacro)
@@ -12,5 +12,13 @@
   <!-- =============== Link & Joint =============== -->
   <!-- Base -->
-  <link name="base_link"/>
+  <link name="base_link">
+    <inertial>
+      <origin xyz="0 0 0"/>
+      <mass value="0.0001"/>
+      <inertia ixx="0.00001" ixy="0" ixz="0"
+                         iyy="0.00001" iyz="0"
+                                 izz="0.00001" />
+    </inertial>
+  </link>
   <xacro:base_v0 parent="base_link">
 	<origin xyz="0 0 0.06"/>
@@ -44,4 +52,11 @@
   </joint>
   <link name="camera_link">
+    <inertial>
+      <origin xyz="0 0 0"/>
+      <mass value="0.0001"/>
+      <inertia ixx="0.00001" ixy="0" ixz="0"
+                         iyy="0.00001" iyz="0"
+                                 izz="0.00001" />
+    </inertial>
   </link>
   <joint name="armor1_joint" type="fixed">

File: colcon_ws/src/sample_robot_description/urdf/wheel/wheel_100mm.urdf.xacro (robot description, xacro)
@@ -60,5 +60,5 @@
         <!-- Links without mass cannot be used in gazebo. -->
         <mass value="0.001"/>
-        <inertia ixx="0" ixy="0" ixz="0" iyy="0" iyz="0" izz="0.00001"/>
+        <inertia ixx="0.00001" ixy="0" ixz="0" iyy="0.00001" iyz="0" izz="0.00001"/>
       </inertial>
     </link>
