Commit message: [change] 引っかからないようにフレームをつける [add] 俯瞰カメラを練習用につける [add] 速度を変えられるようにする [add] フィールド全体を覆う壁を追加

File: colcon_ws/src/sample_robot_description/isaac/sample_robot.isaac.xacro (robot description, xacro)
@@ -19,5 +19,22 @@
           <far>300</far>
         </clip>
-        <update_rate>5.0</update_rate>
+        <update_rate>10.0</update_rate>
+      </sensor>
+      <sensor name="top_view_camera_link" type="camera">
+        <topic>image_raw</topic>
+        <horizontal_fov_rad>0.523599</horizontal_fov_rad>
+        <horizontal_focal_length>30</horizontal_focal_length> <!-- optical parameter -->
+        <vertical_focal_length>30</vertical_focal_length> <!-- optical parameter -->
+        <focus_distance>10</focus_distance> <!-- distance for clear image -->
+        <projection>perspective</projection> <!-- perspective or orthgonal -->
+        <image>
+           <width>180</width>
+           <height>180</height>
+        </image>
+        <clip>
+          <near>5.0</near>
+          <far>15</far>
+        </clip>
+        <update_rate>10.0</update_rate>
       </sensor>
       <sensor name="armor1_link" type="contact">

File: colcon_ws/src/sample_robot_description/robots/sample_robot_1.urdf.xacro (robot description, xacro)
@@ -60,4 +60,18 @@
     </inertial>
   </link>
+  <joint name="top_view_camera_joint" type="fixed">
+    <parent link="base_link"/>
+    <child  link="top_view_camera_link"/>
+    <origin xyz="0.0 0 10.0" rpy="0 ${pi/2} 0"/>
+  </joint>
+  <link name="top_view_camera_link">
+    <inertial>
+      <origin xyz="0 0 0"/>
+      <mass value="0.0001"/>
+      <inertia ixx="0.00001" ixy="0" ixz="0"
+                         iyy="0.00001" iyz="0"
+                                 izz="0.00001" />
+    </inertial>
+  </link>
   <joint name="armor1_joint" type="fixed">
     <parent link="base_link"/>
@@ -70,9 +84,9 @@
         <box size="0.01 0.15 0.15" />
       </geometry>
-      <material name="white"/>
+      <material name="light_blue"/>
     </visual>
     <collision>
       <geometry>
-        <box size="0.1 0.3 0.3" />
+        <box size="0.01 0.15 0.15" />
       </geometry>
     </collision>
@@ -95,9 +109,9 @@
         <box size="0.01 0.15 0.15" />
       </geometry>
-      <material name="white"/>
+      <material name="light_blue"/>
     </visual>
     <collision>
       <geometry>
-        <box size="0.1 0.3 0.3" />
+        <box size="0.01 0.15 0.15" />
       </geometry>
     </collision>
@@ -120,9 +134,9 @@
         <box size="0.01 0.15 0.15" />
       </geometry>
-      <material name="white"/>
+      <material name="light_blue"/>
     </visual>
     <collision>
       <geometry>
-        <box size="0.1 0.3 0.3" />
+        <box size="0.01 0.15 0.15" />
       </geometry>
     </collision>
@@ -145,9 +159,9 @@
         <box size="0.01 0.15 0.15" />
       </geometry>
-      <material name="white"/>
+      <material name="light_blue"/>
     </visual>
     <collision>
       <geometry>
-        <box size="0.1 0.3 0.3" />
+        <box size="0.01 0.15 0.15" />
       </geometry>
     </collision>

File: colcon_ws/src/sample_robot_description/robots/sample_robot_2.urdf.xacro (robot description, xacro)
@@ -60,4 +60,18 @@
     </inertial>
   </link>
+  <joint name="top_view_camera_joint" type="fixed">
+    <parent link="base_link"/>
+    <child  link="top_view_camera_link"/>
+    <origin xyz="0.0 0 10.0" rpy="0 ${pi/2} 0"/>
+  </joint>
+  <link name="top_view_camera_link">
+    <inertial>
+      <origin xyz="0 0 0"/>
+      <mass value="0.0001"/>
+      <inertia ixx="0.00001" ixy="0" ixz="0"
+                         iyy="0.00001" iyz="0"
+                                 izz="0.00001" />
+    </inertial>
+  </link>
   <joint name="armor1_joint" type="fixed">
     <parent link="base_link"/>
@@ -70,9 +84,9 @@
         <box size="0.01 0.15 0.15" />
       </geometry>
-      <material name="white"/>
+      <material name="light_red"/>
     </visual>
     <collision>
       <geometry>
-        <box size="0.1 0.3 0.3" />
+        <box size="0.01 0.15 0.15" />
       </geometry>
     </collision>
@@ -95,9 +109,9 @@
         <box size="0.01 0.15 0.15" />
       </geometry>
-      <material name="white"/>
+      <material name="light_red"/>
     </visual>
     <collision>
       <geometry>
-        <box size="0.1 0.3 0.3" />
+        <box size="0.01 0.15 0.15" />
       </geometry>
     </collision>
@@ -120,9 +134,9 @@
         <box size="0.01 0.15 0.15" />
       </geometry>
-      <material name="white"/>
+      <material name="light_red"/>
     </visual>
     <collision>
       <geometry>
-        <box size="0.1 0.3 0.3" />
+        <box size="0.01 0.15 0.15" />
       </geometry>
     </collision>
@@ -145,9 +159,9 @@
         <box size="0.01 0.15 0.15" />
       </geometry>
-      <material name="white"/>
+      <material name="light_red"/>
     </visual>
     <collision>
       <geometry>
-        <box size="0.1 0.3 0.3" />
+        <box size="0.01 0.15 0.15" />
       </geometry>
     </collision>

File: colcon_ws/src/sample_robot_description/robots/sample_robot_3.urdf.xacro (robot description, xacro)
@@ -60,4 +60,18 @@
     </inertial>
   </link>
+  <joint name="top_view_camera_joint" type="fixed">
+    <parent link="base_link"/>
+    <child  link="top_view_camera_link"/>
+    <origin xyz="0.0 0 10.0" rpy="0 ${pi/2} 0"/>
+  </joint>
+  <link name="top_view_camera_link">
+    <inertial>
+      <origin xyz="0 0 0"/>
+      <mass value="0.0001"/>
+      <inertia ixx="0.00001" ixy="0" ixz="0"
+                         iyy="0.00001" iyz="0"
+                                 izz="0.00001" />
+    </inertial>
+  </link>
   <joint name="armor1_joint" type="fixed">
     <parent link="base_link"/>
@@ -70,9 +84,9 @@
         <box size="0.01 0.15 0.15" />
       </geometry>
-      <material name="white"/>
+      <material name="light_blue"/>
     </visual>
     <collision>
       <geometry>
-        <box size="0.1 0.3 0.3" />
+        <box size="0.01 0.15 0.15" />
       </geometry>
     </collision>
@@ -95,9 +109,9 @@
         <box size="0.01 0.15 0.15" />
       </geometry>
-      <material name="white"/>
+      <material name="light_blue"/>
     </visual>
     <collision>
       <geometry>
-        <box size="0.1 0.3 0.3" />
+        <box size="0.01 0.15 0.15" />
       </geometry>
     </collision>
@@ -120,9 +134,9 @@
         <box size="0.01 0.15 0.15" />
       </geometry>
-      <material name="white"/>
+      <material name="light_blue"/>
     </visual>
     <collision>
       <geometry>
-        <box size="0.1 0.3 0.3" />
+        <box size="0.01 0.15 0.15" />
       </geometry>
     </collision>
@@ -145,9 +159,9 @@
         <box size="0.01 0.15 0.15" />
       </geometry>
-      <material name="white"/>
+      <material name="light_blue"/>
     </visual>
     <collision>
       <geometry>
-        <box size="0.1 0.3 0.3" />
+        <box size="0.01 0.15 0.15" />
       </geometry>
     </collision>

File: colcon_ws/src/sample_robot_description/robots/sample_robot_4.urdf.xacro (robot description, xacro)
@@ -60,4 +60,18 @@
     </inertial>
   </link>
+  <joint name="top_view_camera_joint" type="fixed">
+    <parent link="base_link"/>
+    <child  link="top_view_camera_link"/>
+    <origin xyz="0.0 0 10.0" rpy="0 ${pi/2} 0"/>
+  </joint>
+  <link name="top_view_camera_link">
+    <inertial>
+      <origin xyz="0 0 0"/>
+      <mass value="0.0001"/>
+      <inertia ixx="0.00001" ixy="0" ixz="0"
+                         iyy="0.00001" iyz="0"
+                                 izz="0.00001" />
+    </inertial>
+  </link>
   <joint name="armor1_joint" type="fixed">
     <parent link="base_link"/>
@@ -70,9 +84,9 @@
         <box size="0.01 0.15 0.15" />
       </geometry>
-      <material name="white"/>
+      <material name="orange"/>
     </visual>
     <collision>
       <geometry>
-        <box size="0.6 0.6 0.02" />
+        <box size="0.01 0.15 0.15" />
       </geometry>
     </collision>
@@ -95,9 +109,9 @@
         <box size="0.01 0.15 0.15" />
       </geometry>
-      <material name="white"/>
+      <material name="orange"/>
     </visual>
     <collision>
       <geometry>
-        <box size="0.6 0.6 0.02" />
+        <box size="0.01 0.15 0.15" />
       </geometry>
     </collision>
@@ -120,9 +134,9 @@
         <box size="0.01 0.15 0.15" />
       </geometry>
-      <material name="white"/>
+      <material name="orange"/>
     </visual>
     <collision>
       <geometry>
-        <box size="0.6 0.6 0.02" />
+        <box size="0.01 0.15 0.15" />
       </geometry>
     </collision>
@@ -145,9 +159,9 @@
         <box size="0.01 0.15 0.15" />
       </geometry>
-      <material name="white"/>
+      <material name="orange"/>
     </visual>
     <collision>
       <geometry>
-        <box size="0.6 0.6 0.02" />
+        <box size="0.01 0.15 0.15" />
       </geometry>
     </collision>

File: colcon_ws/src/sample_robot_description/robots/sample_robot_5.urdf.xacro (robot description, xacro)
@@ -60,4 +60,18 @@
     </inertial>
   </link>
+  <joint name="top_view_camera_joint" type="fixed">
+    <parent link="base_link"/>
+    <child  link="top_view_camera_link"/>
+    <origin xyz="0.0 0 10.0" rpy="0 ${pi/2} 0"/>
+  </joint>
+  <link name="top_view_camera_link">
+    <inertial>
+      <origin xyz="0 0 0"/>
+      <mass value="0.0001"/>
+      <inertia ixx="0.00001" ixy="0" ixz="0"
+                         iyy="0.00001" iyz="0"
+                                 izz="0.00001" />
+    </inertial>
+  </link>
   <joint name="armor1_joint" type="fixed">
     <parent link="base_link"/>
@@ -70,9 +84,9 @@
         <box size="0.01 0.15 0.15" />
       </geometry>
-      <material name="white"/>
+      <material name="purple"/>
     </visual>
     <collision>
       <geometry>
-        <box size="0.6 0.6 0.02" />
+        <box size="0.01 0.15 0.15" />
       </geometry>
     </collision>
@@ -95,9 +109,9 @@
         <box size="0.01 0.15 0.15" />
       </geometry>
-      <material name="white"/>
+      <material name="purple"/>
     </visual>
     <collision>
       <geometry>
-        <box size="0.6 0.6 0.02" />
+        <box size="0.01 0.15 0.15" />
       </geometry>
     </collision>
@@ -120,9 +134,9 @@
         <box size="0.01 0.15 0.15" />
       </geometry>
-      <material name="white"/>
+      <material name="purple"/>
     </visual>
     <collision>
       <geometry>
-        <box size="0.6 0.6 0.02" />
+        <box size="0.01 0.15 0.15" />
       </geometry>
     </collision>
@@ -145,9 +159,9 @@
         <box size="0.01 0.15 0.15" />
       </geometry>
-      <material name="white"/>
+      <material name="purple"/>
     </visual>
     <collision>
       <geometry>
-        <box size="0.6 0.6 0.02" />
+        <box size="0.01 0.15 0.15" />
       </geometry>
     </collision>

File: colcon_ws/src/sample_robot_description/robots/sample_robot_6.urdf.xacro (robot description, xacro)
@@ -60,4 +60,18 @@
     </inertial>
   </link>
+  <joint name="top_view_camera_joint" type="fixed">
+    <parent link="base_link"/>
+    <child  link="top_view_camera_link"/>
+    <origin xyz="0.0 0 10.0" rpy="0 ${pi/2} 0"/>
+  </joint>
+  <link name="top_view_camera_link">
+    <inertial>
+      <origin xyz="0 0 0"/>
+      <mass value="0.0001"/>
+      <inertia ixx="0.00001" ixy="0" ixz="0"
+                         iyy="0.00001" iyz="0"
+                                 izz="0.00001" />
+    </inertial>
+  </link>
   <joint name="armor1_joint" type="fixed">
     <parent link="base_link"/>
@@ -70,9 +84,9 @@
         <box size="0.01 0.15 0.15" />
       </geometry>
-      <material name="white"/>
+      <material name="yellow"/>
     </visual>
     <collision>
       <geometry>
-        <box size="0.6 0.6 0.02" />
+        <box size="0.01 0.15 0.15" />
       </geometry>
     </collision>
@@ -95,9 +109,9 @@
         <box size="0.01 0.15 0.15" />
       </geometry>
-      <material name="white"/>
+      <material name="yellow"/>
     </visual>
     <collision>
       <geometry>
-        <box size="0.6 0.6 0.02" />
+        <box size="0.01 0.15 0.15" />
       </geometry>
     </collision>
@@ -120,9 +134,9 @@
         <box size="0.01 0.15 0.15" />
       </geometry>
-      <material name="white"/>
+      <material name="yellow"/>
     </visual>
     <collision>
       <geometry>
-        <box size="0.6 0.6 0.02" />
+        <box size="0.01 0.15 0.15" />
       </geometry>
     </collision>
@@ -145,9 +159,9 @@
         <box size="0.01 0.15 0.15" />
       </geometry>
-      <material name="white"/>
+      <material name="yellow"/>
     </visual>
     <collision>
       <geometry>
-        <box size="0.6 0.6 0.02" />
+        <box size="0.01 0.15 0.15" />
       </geometry>
     </collision>

File: colcon_ws/src/sample_robot_description/robots/sample_robot_7.urdf.xacro (robot description, xacro)
@@ -60,4 +60,18 @@
     </inertial>
   </link>
+  <joint name="top_view_camera_joint" type="fixed">
+    <parent link="base_link"/>
+    <child  link="top_view_camera_link"/>
+    <origin xyz="0.0 0 10.0" rpy="0 ${pi/2} 0"/>
+  </joint>
+  <link name="top_view_camera_link">
+    <inertial>
+      <origin xyz="0 0 0"/>
+      <mass value="0.0001"/>
+      <inertia ixx="0.00001" ixy="0" ixz="0"
+                         iyy="0.00001" iyz="0"
+                                 izz="0.00001" />
+    </inertial>
+  </link>
   <joint name="armor1_joint" type="fixed">
     <parent link="base_link"/>
@@ -70,9 +84,9 @@
         <box size="0.01 0.15 0.15" />
       </geometry>
-      <material name="white"/>
+      <material name="blue_green"/>
     </visual>
     <collision>
       <geometry>
-        <box size="0.6 0.6 0.02" />
+        <box size="0.01 0.15 0.15" />
       </geometry>
     </collision>
@@ -95,9 +109,9 @@
         <box size="0.01 0.15 0.15" />
       </geometry>
-      <material name="white"/>
+      <material name="blue_green"/>
     </visual>
     <collision>
       <geometry>
-        <box size="0.6 0.6 0.02" />
+        <box size="0.01 0.15 0.15" />
       </geometry>
     </collision>
@@ -120,9 +134,9 @@
         <box size="0.01 0.15 0.15" />
       </geometry>
-      <material name="white"/>
+      <material name="blue_green"/>
     </visual>
     <collision>
       <geometry>
-        <box size="0.6 0.6 0.02" />
+        <box size="0.01 0.15 0.15" />
       </geometry>
     </collision>
@@ -145,9 +159,9 @@
         <box size="0.01 0.15 0.15" />
       </geometry>
-      <material name="white"/>
+      <material name="blue_green"/>
     </visual>
     <collision>
       <geometry>
-        <box size="0.6 0.6 0.02" />
+        <box size="0.01 0.15 0.15" />
       </geometry>
     </collision>

File: colcon_ws/src/sample_robot_description/robots/sample_robot_8.urdf.xacro (robot description, xacro)
@@ -60,4 +60,18 @@
     </inertial>
   </link>
+  <joint name="top_view_camera_joint" type="fixed">
+    <parent link="base_link"/>
+    <child  link="top_view_camera_link"/>
+    <origin xyz="0.0 0 10.0" rpy="0 ${pi/2} 0"/>
+  </joint>
+  <link name="top_view_camera_link">
+    <inertial>
+      <origin xyz="0 0 0"/>
+      <mass value="0.0001"/>
+      <inertia ixx="0.00001" ixy="0" ixz="0"
+                         iyy="0.00001" iyz="0"
+                                 izz="0.00001" />
+    </inertial>
+  </link>
   <joint name="armor1_joint" type="fixed">
     <parent link="base_link"/>
@@ -70,9 +84,9 @@
         <box size="0.01 0.15 0.15" />
       </geometry>
-      <material name="white"/>
+      <material name="yellow_green"/>
     </visual>
     <collision>
       <geometry>
-        <box size="0.6 0.6 0.02" />
+        <box size="0.01 0.15 0.15" />
       </geometry>
     </collision>
@@ -95,9 +109,9 @@
         <box size="0.01 0.15 0.15" />
       </geometry>
-      <material name="white"/>
+      <material name="yellow_green"/>
     </visual>
     <collision>
       <geometry>
-        <box size="0.6 0.6 0.02" />
+        <box size="0.01 0.15 0.15" />
       </geometry>
     </collision>
@@ -120,9 +134,9 @@
         <box size="0.01 0.15 0.15" />
       </geometry>
-      <material name="white"/>
+      <material name="yellow_green"/>
     </visual>
     <collision>
       <geometry>
-        <box size="0.6 0.6 0.02" />
+        <box size="0.01 0.15 0.15" />
       </geometry>
     </collision>
@@ -145,9 +159,9 @@
         <box size="0.01 0.15 0.15" />
       </geometry>
-      <material name="white"/>
+      <material name="yellow_green"/>
     </visual>
     <collision>
       <geometry>
-        <box size="0.6 0.6 0.02" />
+        <box size="0.01 0.15 0.15" />
       </geometry>
     </collision>

File: colcon_ws/src/sample_robot_description/ros2_control/sample_robot.ros2_control.xacro (robot description, xacro)
@@ -18,6 +18,6 @@
       <joint name="wheel0_shaft_joint">
         <command_interface name="velocity">
-          <param name="min">-6</param>
-          <param name="max">6</param>
+          <param name="min">-100</param>
+          <param name="max">100</param>
         </command_interface>
         <state_interface name="position">
@@ -29,6 +29,6 @@
       <joint name="wheel1_shaft_joint">
         <command_interface name="velocity">
-          <param name="min">-6</param>
-          <param name="max">6</param>
+          <param name="min">-100</param>
+          <param name="max">100</param>
         </command_interface>
         <state_interface name="position">
@@ -40,6 +40,6 @@
       <joint name="wheel2_shaft_joint">
         <command_interface name="velocity">
-          <param name="min">-6</param>
-          <param name="max">6</param>
+          <param name="min">-100</param>
+          <param name="max">100</param>
         </command_interface>
         <state_interface name="position">
@@ -51,6 +51,6 @@
       <joint name="wheel3_shaft_joint">
         <command_interface name="velocity">
-          <param name="min">-6</param>
-          <param name="max">6</param>
+          <param name="min">-100</param>
+          <param name="max">100</param>
         </command_interface>
         <state_interface name="position">

File: colcon_ws/src/sample_robot_description/urdf/base/base.urdf.xacro (robot description, xacro)
@@ -28,4 +28,104 @@
           </inertial>
         </link>
+        <joint name="bumper1_joint" type="fixed">
+          <parent link="${parent}"/>
+          <child  link="bumper1_link"/>
+          <origin xyz="-0.45 0.0 0.10" rpy="0 0 0"/>
+        </joint>
+        <link name="bumper1_link">
+          <visual>
+            <geometry>
+              <box size="0.01 0.9 0.10" />
+            </geometry>
+            <material name="white"/>
+          </visual>
+          <collision>
+            <geometry>
+              <box size="0.01 0.9 0.10" />
+            </geometry>
+          </collision>
+          <inertial>
+            <origin xyz="0 0 0"/>
+            <mass value="0.4"/>
+            <inertia ixx="0.1" ixy="0" ixz="0"
+                               iyy="0.1" iyz="0"
+                                         izz="0.1" />
+          </inertial>
+        </link>
+        <joint name="bumper2_joint" type="fixed">
+          <parent link="${parent}"/>
+          <child  link="bumper2_link"/>
+          <origin xyz="0.0 0.45 0.10" rpy="0 0 0"/>
+        </joint>
+        <link name="bumper2_link">
+          <visual>
+            <geometry>
+              <box size="0.9 0.01 0.10" />
+            </geometry>
+            <material name="white"/>
+          </visual>
+          <collision>
+            <geometry>
+              <box size="0.9 0.01 0.10" />
+            </geometry>
+          </collision>
+          <inertial>
+            <origin xyz="0 0 0"/>
+            <mass value="0.4"/>
+            <inertia ixx="0.1" ixy="0" ixz="0"
+                               iyy="0.1" iyz="0"
+                                         izz="0.1" />
+          </inertial>
+        </link>
+        <joint name="bumper3_joint" type="fixed">
+          <parent link="${parent}"/>
+          <child  link="bumper3_link"/>
+          <origin xyz="0.0 -0.45 0.10" rpy="0 0 0"/>
+        </joint>
+        <link name="bumper3_link">
+          <visual>
+            <geometry>
+              <box size="0.9 0.01 0.10" />
+            </geometry>
+            <material name="white"/>
+          </visual>
+          <collision>
+            <geometry>
+              <box size="0.9 0.01 0.10" />
+            </geometry>
+          </collision>
+          <inertial>
+            <origin xyz="0 0 0"/>
+            <mass value="0.4"/>
+            <inertia ixx="0.1" ixy="0" ixz="0"
+                               iyy="0.1" iyz="0"
+                                         izz="0.1" />
+          </inertial>
+        </link>
+        <joint name="bumper4_joint" type="fixed">
+          <parent link="${parent}"/>
+          <child  link="bumper4_link"/>
+          <origin xyz="0.45 0.0 0.10" rpy="0 0 0"/>
+        </joint>
+        <link name="bumper4_link">
+          <visual>
+            <geometry>
+              <box size="0.01 0.9 0.10" />
+            </geometry>
+            <material name="white"/>
+          </visual>
+          <collision>
+            <geometry>
+              <box size="0.01 0.9 0.10" />
+            </geometry>
+          </collision>
+          <inertial>
+            <origin xyz="0 0 0"/>
+            <mass value="0.4"/>
+            <inertia ixx="0.1" ixy="0" ixz="0"
+                               iyy="0.1" iyz="0"
+                                         izz="0.1" />
+          </inertial>
+        </link>
   </xacro:macro>
 </robot>

File: colcon_ws/src/sample_robot_description/urdf/common.xacro (robot description, xacro)
@@ -23,9 +23,33 @@
   </material>
   <material name="light_red">
-    <color rgba="1.0 0.5 0.5 1.0"/>
+    <color rgba="1.0 0.5 0.5 0.6"/>
+    <isaac_rigid_body static_friction="1.0" dynamic_friction="1.0"/>
+  </material>
+  <material name="orange">
+    <color rgba="1.0 0.5 0.0 1.0"/>
     <isaac_rigid_body static_friction="1.0" dynamic_friction="1.0"/>
   </material>
   <material name="yellow">
-    <color rgba="0 1.0 1.0 1.0"/>
+    <color rgba="1.0 1.0 0.0 1.0"/>
+    <isaac_rigid_body static_friction="1.0" dynamic_friction="1.0"/>
+  </material>
+  <material name="yellow_green">
+    <color rgba="0.5 1.0 0.0 1.0"/>
+    <isaac_rigid_body static_friction="1.0" dynamic_friction="1.0"/>
+  </material>
+  <material name="blue">
+    <color rgba="0.0 0.0 1.0 1.0"/>
+    <isaac_rigid_body static_friction="1.0" dynamic_friction="1.0"/>
+  </material>
+  <material name="light_blue">
+    <color rgba="0.5 0.5 1.0 0.6"/>
+    <isaac_rigid_body static_friction="1.0" dynamic_friction="1.0"/>
+  </material>
+  <material name="purple">
+    <color rgba="1.0 0.0 1.0 1.0"/>
+    <isaac_rigid_body static_friction="1.0" dynamic_friction="1.0"/>
+  </material>
+  <material name="blue_green">
+    <color rgba="0.0 1.0 0.5 1.0"/>
     <isaac_rigid_body static_friction="1.0" dynamic_friction="1.0"/>
   </material>
